File: hybrid.brd (EAGLE design)
At the start: 161.3 x 168.9 mm, 125 parts, among them IC1 TL071P, IC2 TL071P, IC3 LM317MABT, IC4 LM317MABT, J1 RCJ-21XXMILL, J2 NRJ3HF-1, J3 703W-00/54, Q1 BC560KINKED, Q10 BC560KINKED, Q11 BC560KINKED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

Commit message: Back to gain stage with uncompensated PSN
Connections:
- net GND: now also C1.1, C11.1
- net HT: no longer C1.1, C11.1
Routing:
- net HT: track 258.0 -> 227.5 mm
Changed lines of the file:
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@@
 <via x="22.86" y="15.24" extent="1-16" drill="0.8"/>
 <via x="19.05" y="11.43" extent="1-16" drill="0.8"/>
+<contactref element="C1" pad="1"/>
+<contactref element="C11" pad="1"/>
 </signal>
 <signal name="CAT_L">
@@
 <wire x1="70.33" y1="62.23" x2="73.66" y2="62.23" width="1.778" layer="1"/>
 <wire x1="112.55" y1="62.23" x2="109.22" y2="62.23" width="1.778" layer="1"/>
-<contactref element="C1" pad="1"/>
-<contactref element="C11" pad="1"/>
-<wire x1="58.42" y1="58.42" x2="73.66" y2="58.42" width="0.8128" layer="1"/>
-<wire x1="124.46" y1="58.42" x2="109.22" y2="58.42" width="0.8128" layer="1"/>
 <via x="54.61" y="96.52" extent="1-16" drill="0.8"/>
 <wire x1="64.77" y1="80.01" x2="67.31" y2="80.01" width="1.778" layer="1"/>

Commit message: PDFs
Routing:
- net GND: vias 52 -> 63
Changed lines of the file:
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@@
 <?xml version="1.0" encoding="utf-8"?>
 <!DOCTYPE eagle SYSTEM "eagle.dtd">
-<eagle version="8.0.0">
+<eagle version="8.0.1">
 <drawing>
 <settings>
@@
 <wire x1="0" y1="36.83" x2="22.86" y2="36.83" width="0.8128" layer="42"/>
 <dimension x1="161.29" y1="0" x2="161.29" y2="168.91" x3="180.34" y3="84.455" textsize="1.27" layer="47" dtype="vertical"/>
-<dimension x1="0" y1="168.91" x2="124.46" y2="168.91" x3="62.23" y3="187.96" textsize="1.27" layer="47" dtype="horizontal"/>
+<dimension x1="0" y1="168.91" x2="161.29" y2="168.91" x3="80.645" y3="186.69" textsize="1.27" layer="47" dtype="horizontal"/>
 </plain>
 <attributes>
@@
 <wire x1="87.63" y1="88.9" x2="87.63" y2="91.44" width="0.8128" layer="1"/>
 <contactref element="H4" pad="B3,2"/>
-<via x="52.07" y="7.62" extent="1-16" drill="0.8"/>
-<via x="57.15" y="7.62" extent="1-16" drill="0.8"/>
-<via x="62.23" y="7.62" extent="1-16" drill="0.8"/>
-<via x="50.8" y="16.51" extent="1-16" drill="0.8"/>
-<via x="50.8" y="21.59" extent="1-16" drill="0.8"/>
-<via x="57.15" y="21.59" extent="1-16" drill="0.8"/>
-<via x="57.15" y="16.51" extent="1-16" drill="0.8"/>
-<via x="62.23" y="21.59" extent="1-16" drill="0.8"/>
-<via x="66.04" y="24.13" extent="1-16" drill="0.8"/>
-<via x="71.12" y="24.13" extent="1-16" drill="0.8"/>
-<via x="125.73" y="7.62" extent="1-16" drill="0.8"/>
-<via x="120.65" y="7.62" extent="1-16" drill="0.8"/>
-<via x="130.81" y="7.62" extent="1-16" drill="0.8"/>
-<via x="125.73" y="16.51" extent="1-16" drill="0.8"/>
-<via x="125.73" y="21.59" extent="1-16" drill="0.8"/>
-<via x="130.81" y="21.59" extent="1-16" drill="0.8"/>
-<via x="120.65" y="21.59" extent="1-16" drill="0.8"/>
-<via x="120.65" y="16.51" extent="1-16" drill="0.8"/>
-<via x="127" y="30.48" extent="1-16" drill="0.8"/>
-<via x="120.65" y="30.48" extent="1-16" drill="0.8"/>
-<via x="86.36" y="3.81" extent="1-16" drill="0.8"/>
-<via x="97.79" y="3.81" extent="1-16" drill="0.8"/>
-<via x="91.44" y="17.78" extent="1-16" drill="0.8"/>
-<via x="91.44" y="22.86" extent="1-16" drill="0.8"/>
-<via x="91.44" y="27.94" extent="1-16" drill="0.8"/>
-<via x="91.44" y="33.02" extent="1-16" drill="0.8"/>
-<via x="99.06" y="16.51" extent="1-16" drill="0.8"/>
-<via x="101.6" y="19.05" extent="1-16" drill="0.8"/>
-<via x="82.55" y="16.51" extent="1-16" drill="0.8"/>
-<via x="80.01" y="19.05" extent="1-16" drill="0.8"/>
-<via x="82.55" y="24.13" extent="1-16" drill="0.8"/>
-<via x="100.33" y="24.13" extent="1-16" drill="0.8"/>
-<via x="81.28" y="73.66" extent="1-16" drill="0.8"/>
-<via x="81.28" y="67.31" extent="1-16" drill="0.8"/>
-<via x="101.6" y="67.31" extent="1-16" drill="0.8"/>
-<via x="101.6" y="73.66" extent="1-16" drill="0.8"/>
-<via x="101.6" y="70.485" extent="1-16" drill="0.8"/>
-<via x="81.28" y="70.485" extent="1-16" drill="0.8"/>
-<via x="144.78" y="8.89" extent="1-16" drill="0.8"/>
-<via x="142.24" y="7.62" extent="1-16" drill="0.8"/>
-<via x="87.63" y="73.66" extent="1-16" drill="0.8"/>
-<via x="95.25" y="73.66" extent="1-16" drill="0.8"/>
-<via x="86.995" y="67.31" extent="1-16" drill="0.8"/>
-<via x="95.885" y="67.31" extent="1-16" drill="0.8"/>
+<via x="52.07" y="7.62" extent="1-16" drill="0.6"/>
+<via x="57.15" y="7.62" extent="1-16" drill="0.6"/>
+<via x="62.23" y="7.62" extent="1-16" drill="0.6"/>
+<via x="52.07" y="16.51" extent="1-16" drill="0.6"/>
+<via x="52.07" y="21.59" extent="1-16" drill="0.6"/>
+<via x="57.15" y="21.59" extent="1-16" drill="0.6"/>
+<via x="57.15" y="16.51" extent="1-16" drill="0.6"/>
+<via x="62.23" y="21.59" extent="1-16" drill="0.6"/>
+<via x="66.04" y="24.13" extent="1-16" drill="0.6"/>
+<via x="71.12" y="24.13" extent="1-16" drill="0.6"/>
+<via x="125.73" y="7.62" extent="1-16" drill="0.6"/>
+<via x="120.65" y="7.62" extent="1-16" drill="0.6"/>
+<via x="130.81" y="7.62" extent="1-16" drill="0.6"/>
+<via x="125.73" y="16.51" extent="1-16" drill="0.6"/>
+<via x="125.73" y="21.59" extent="1-16" drill="0.6"/>
+<via x="130.81" y="21.59" extent="1-16" drill="0.6"/>
+<via x="120.65" y="21.59" extent="1-16" drill="0.6"/>
+<via x="120.65" y="16.51" extent="1-16" drill="0.6"/>
+<via x="127" y="30.48" extent="1-16" drill="0.6"/>
+<via x="120.65" y="30.48" extent="1-16" drill="0.6"/>
+<via x="86.36" y="3.81" extent="1-16" drill="0.6"/>
+<via x="97.79" y="3.81" extent="1-16" drill="0.6"/>
+<via x="91.44" y="17.78" extent="1-16" drill="0.6"/>
+<via x="91.44" y="22.86" extent="1-16" drill="0.6"/>
+<via x="91.44" y="27.94" extent="1-16" drill="0.6"/>
+<via x="91.44" y="33.02" extent="1-16" drill="0.6"/>
+<via x="99.06" y="16.51" extent="1-16" drill="0.6"/>
+<via x="101.6" y="19.05" extent="1-16" drill="0.6"/>
+<via x="82.55" y="16.51" extent="1-16" drill="0.6"/>
+<via x="80.01" y="19.05" extent="1-16" drill="0.6"/>
+<via x="82.55" y="24.13" extent="1-16" drill="0.6"/>
+<via x="100.33" y="24.13" extent="1-16" drill="0.6"/>
+<via x="81.28" y="73.66" extent="1-16" drill="0.6"/>
+<via x="81.28" y="67.31" extent="1-16" drill="0.6"/>
+<via x="101.6" y="67.31" extent="1-16" drill="0.6"/>
+<via x="101.6" y="73.66" extent="1-16" drill="0.6"/>
+<via x="101.6" y="70.485" extent="1-16" drill="0.6"/>
+<via x="81.28" y="70.485" extent="1-16" drill="0.6"/>
+<via x="144.78" y="8.89" extent="1-16" drill="0.6"/>
+<via x="142.24" y="7.62" extent="1-16" drill="0.6"/>
+<via x="87.63" y="73.66" extent="1-16" drill="0.6"/>
+<via x="95.25" y="73.66" extent="1-16" drill="0.6"/>
+<via x="86.995" y="67.31" extent="1-16" drill="0.6"/>
+<via x="95.885" y="67.31" extent="1-16" drill="0.6"/>
 <contactref element="D7" pad="K"/>
-<via x="36.83" y="8.89" extent="1-16" drill="0.8"/>
-<via x="34.29" y="11.43" extent="1-16" drill="0.8"/>
-<via x="34.29" y="16.51" extent="1-16" drill="0.8"/>
-<via x="34.29" y="20.32" extent="1-16" drill="0.8"/>
-<via x="23.495" y="10.16" extent="1-16" drill="0.8"/>
-<via x="22.86" y="15.24" extent="1-16" drill="0.8"/>
-<via x="19.05" y="11.43" extent="1-16" drill="0.8"/>
+<via x="36.83" y="8.89" extent="1-16" drill="0.6"/>
+<via x="34.29" y="11.43" extent="1-16" drill="0.6"/>
+<via x="34.29" y="16.51" extent="1-16" drill="0.6"/>
+<via x="34.29" y="20.32" extent="1-16" drill="0.6"/>
+<via x="23.495" y="10.16" extent="1-16" drill="0.6"/>
+<via x="22.86" y="15.24" extent="1-16" drill="0.6"/>
+<via x="19.05" y="11.43" extent="1-16" drill="0.6"/>
 <contactref element="C1" pad="1"/>
 <contactref element="C11" pad="1"/>
+<via x="41.275" y="15.24" extent="1-16" drill="0.6"/>
+<via x="44.45" y="21.59" extent="1-16" drill="0.6"/>
+<via x="87.63" y="16.51" extent="1-16" drill="0.6"/>
+<via x="111.76" y="21.59" extent="1-16" drill="0.6"/>
+<via x="116.84" y="21.59" extent="1-16" drill="0.6"/>
+<via x="133.985" y="16.51" extent="1-16" drill="0.6"/>
+<via x="140.335" y="16.51" extent="1-16" drill="0.6"/>
+<via x="139.7" y="21.59" extent="1-16" drill="0.6"/>
+<via x="48.26" y="21.59" extent="1-16" drill="0.6"/>
+<via x="65.405" y="16.51" extent="1-16" drill="0.6"/>
+<via x="71.755" y="16.51" extent="1-16" drill="0.6"/>
 </signal>
 <signal name="CAT_L">
