File: hybrid.brd (EAGLE design)
At the start: 161.3 x 168.9 mm, 125 parts, among them IC1 TL071P, IC2 TL071P, IC3 LM317MABT, IC4 LM317MABT, J1 RCJ-21XXMILL, J2 NRJ3HF-1, J3 703W-00/54, Q1 BC560KINKED, Q10 BC560KINKED, Q11 BC560KINKED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

Commit message: Minor tweaks
Routing:
- net GND: vias 63 -> 57
Changed lines of the file:
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@@
 <wire x1="33.02" y1="87.63" x2="0" y2="87.63" width="2.54" layer="41"/>
 <wire x1="33.02" y1="87.63" x2="0" y2="87.63" width="2.54" layer="42"/>
-<wire x1="0" y1="36.83" x2="22.86" y2="36.83" width="0.8128" layer="41"/>
-<wire x1="0" y1="36.83" x2="22.86" y2="36.83" width="0.8128" layer="42"/>
 <dimension x1="161.29" y1="0" x2="161.29" y2="168.91" x3="180.34" y3="84.455" textsize="1.778" layer="47" dtype="vertical"/>
 <dimension x1="0" y1="168.91" x2="161.29" y2="168.91" x3="80.645" y3="186.69" textsize="1.778" layer="47" dtype="horizontal"/>
@@
 <via x="100.33" y="24.13" extent="1-16" drill="0.6"/>
 <via x="81.28" y="73.66" extent="1-16" drill="0.6"/>
-<via x="81.28" y="67.31" extent="1-16" drill="0.6"/>
-<via x="101.6" y="67.31" extent="1-16" drill="0.6"/>
 <via x="101.6" y="73.66" extent="1-16" drill="0.6"/>
-<via x="101.6" y="70.485" extent="1-16" drill="0.6"/>
-<via x="81.28" y="70.485" extent="1-16" drill="0.6"/>
 <via x="144.78" y="8.89" extent="1-16" drill="0.6"/>
 <via x="142.24" y="7.62" extent="1-16" drill="0.6"/>
 <via x="87.63" y="73.66" extent="1-16" drill="0.6"/>
 <via x="95.25" y="73.66" extent="1-16" drill="0.6"/>
-<via x="86.995" y="67.31" extent="1-16" drill="0.6"/>
-<via x="95.885" y="67.31" extent="1-16" drill="0.6"/>
 <contactref element="D7" pad="K"/>
 <via x="36.83" y="8.89" extent="1-16" drill="0.6"/>
