File: Amp2/hybrid.sch (EAGLE design)
At the start: 122 parts, among them IC1 TL071P, IC2 TL071P, IC3 LM317MABT-OUT, IC4 LM317MABT-OUT, J1 RCJ-21XXMILL, J2 NRJ3HF-1, J3 703W-00/54, Q1 BC560KINKED, Q10 BC560KINKED, Q11 BC560KINKED, Q12 BC560KINKED, Q13 BC556KINKED, Q14 BC550KINKED, Q15 BC550KINKED, Q16 BC560KINKED, Q17 BD140, Q18 BD139, Q19 KSP43, Q2 BC560KINKED, Q3 BC560KINKED, Q4 BC556KINKED, Q5 BC550KINKED, Q6 BC550KINKED, Q7 BC560KINKED, Q8 BD140, Q9 BD139, T1 TR-LP30-1600

Commit message: Improved auto biasing circuit
Parts:
- removed C32: 47uF, my-cap:CAP_POLPTH-8/3.5
- removed H5: MOUNT-HOLE3.2, holes:MOUNT-HOLE3.2
- added C25: 47uF, my-cap:CAP_POLPTH-12/5
- added H1: MOUNT-PAD-ROUND3.2, holes:MOUNT-PAD-ROUND3.2
- added Q20: BD139, transistor-npn:BD139
- added Q21: KSP43, my-tran:KSP43
- C1, C11: value 0.1uF -> 1uF; device SparkFun-Capacitors:CAPPTH -> capacitor-wima:C5/5
- C26: value 47uF -> 10uF; device my-cap:CAP_POLPTH-12/5 -> my-cap:CAP_POLPTH-5/2.5
- C27: device my-cap:CAP_POLPTH-5/2.5 -> my-cap:CAP_POLPTH-6.5/2.5
- C28: value 10uF -> 1uF; device my-cap:CAP_POLPTH-6.5/2.5 -> SparkFun-Capacitors:CAPPTH
- C30: value 1uF -> 47uF; device SparkFun-Capacitors:CAPPTH -> my-cap:CAP_POLPTH-8/3.5
- H4: value MOUNT-PAD-ROUND3.2 -> MOUNT-HOLE3.2; device holes:MOUNT-PAD-ROUND3.2 -> holes:MOUNT-HOLE3.2
- Q1, Q11: value BC560KINKED -> KSP06KINKED; device my-tran:BC560KINKED -> my-tran:KSP06KINKED
- Q10: value BC560KINKED -> BD139; device my-tran:BC560KINKED -> transistor-npn:BD139
- Q13, Q4: value BC556KINKED -> BC560KINKED; device my-tran:BC556KINKED -> my-tran:BC560KINKED
- Q14: value BC550KINKED -> BC560KINKED; device my-tran:BC550KINKED -> my-tran:BC560KINKED
- Q15, Q5: value BC550KINKED -> BC556KINKED; device my-tran:BC550KINKED -> my-tran:BC556KINKED
- Q16, Q7: value BC560KINKED -> BC550KINKED; device my-tran:BC560KINKED -> my-tran:BC550KINKED
- Q17: value BD140 -> BC550KINKED; device transistor-pnp:BD140 -> my-tran:BC550KINKED
- Q18: value BD139 -> BC560KINKED; device transistor-npn:BD139 -> my-tran:BC560KINKED
- Q19: value KSP43 -> BD140; device my-tran:KSP43 -> transistor-pnp:BD140
- Q8: value BD140 -> BC560KINKED; device transistor-pnp:BD140 -> my-tran:BC560KINKED
- Q9: value BD139 -> BD140; device transistor-npn:BD139 -> transistor-pnp:BD140
- R1, R20: value 100k -> 1Meg
- R2, R21: value 1Meg -> 2Meg
- R22, R3: value 100k -> 2Meg
- R24, R5: value 27k -> 5.1k
- renumbered U$1 to LOGO1
Connections:
- new net N$47: Q1.E, R5.2
- new net N$48: Q11.E, R24.2
- net FB_L: now also R1.2; no longer R2.2
- net FB_R: now also R20.2; no longer R21.2
- net GND: now also C25.-, C28.2, C30.-, H1.MOUNT, Q10.E, Q20.E, R22.2, R24.1, R3.2, R5.1; no longer C28.-, C30.2, C32.-, H4.MOUNT, Q18.E, Q9.E, R1.1, R20.1
- net HT: now also C31.+; no longer C32.+
- net ISET_L: now also Q2.C, Q4.B; no longer Q3.B, R5.2
- net ISET_R: now also Q11.C, Q12.C, Q14.B; no longer Q10.C, Q12.B, R24.2
- net N$1: now also Q3.B, Q3.C, Q4.E; no longer Q1.B, Q2.C, Q3.E
- net N$11: now also Q7.E, Q9.C; no longer Q6.E, Q8.C
- net N$12: now also Q6.E, Q8.B; no longer Q5.E, Q7.B
- net N$13: now also Q10.C, Q8.E; no longer Q7.E, Q9.C
- net N$14: now also Q7.C, Q9.B; no longer Q6.C, Q8.B
- net N$15: now also Q10.B, Q8.C; no longer Q7.C, Q9.B
- net N$16: now also Q13.E; no longer Q11.E
- net N$17: now also Q12.B, Q13.B, Q13.C, Q14.E; no longer Q10.B, Q11.B, Q11.C, Q12.E
- net N$2: now also Q3.E; no longer Q2.E
- net N$20: now also Q15.E; no longer Q13.E
- net N$21: now also Q15.C, Q16.C, Q17.B; no longer Q13.C, Q14.C, Q15.B
- net N$22: now also Q16.B; no longer Q14.B
- net N$24: now also Q16.E, Q18.B; no longer Q14.E, Q16.B
- net N$25: now also Q17.E, Q19.C; no longer Q15.E, Q17.C
- net N$26: now also Q18.E, Q20.C; no longer Q16.E, Q18.C
- net N$27: now also Q17.C, Q19.B; no longer Q15.C, Q17.B
- net N$28: now also Q18.C, Q20.B; no longer Q16.C, Q18.B
- net N$29: now also Q1.B; no longer R5.1
- net N$3: now also Q2.E; no longer Q1.E
- net N$30: now also C26.+, C28.1; no longer C27.+, C29.1
- net N$33: now also Q21.C; no longer Q19.C
- net N$34: now also C25.+, Q21.B; no longer C26.+, Q19.B
- net N$35: now also R3.1
- net N$36: now also C27.+, C29.1; no longer C28.+, C30.1
- net N$37: now also Q21.E; no longer Q19.E
- net N$38: now also R1.1; no longer R1.2, R3.1
- net N$39: now also Q12.E; no longer Q10.E
- net N$41: now also C13.2, IC2.-IN, R21.1, R22.1; no longer C13.1, IC2.OUT, R24.1
- net N$42: now also C11.2, IC2.+IN, R20.1; no longer C13.2, IC2.-IN, R21.1
- net N$43: now also C13.1, IC2.OUT, Q11.B; no longer C11.2, IC2.+IN, R20.2, R22.1
- net N$5: now also Q5.E; no longer Q4.E
- net N$7: now also Q6.C, Q7.B; no longer Q4.C, Q6.B
- net N$8: now also Q6.B; no longer Q5.B
- net PL_L: now also Q4.C, Q5.B; no longer Q3.C, Q4.B
- net PL_R: now also Q14.C, Q15.B; no longer Q12.C, Q13.B
- net VCC: now also C30.+, Q19.E, Q9.E, R2.2, R21.2; no longer C31.+, Q17.E, Q8.E, R22.2, R3.2
Other:
- moved on the sheet: C1, C11, C12, C13, C14, C15, C16, C17, C18, C19, C20, C26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

Commit message: Back to toroidal transformer
Parts:
- removed T1: TR-LP30-1600, my-transformers:TR-LP30-1600
- added PAD1, PAD2, PAD3, PAD4: (no value), wirepad:3,81/1,4
Connections:
- removed net N$6: T1.2, T1.3
- removed net N$9: T1.6, T1.7
- net AC_1: now also PAD4.P; no longer T1.8
- net AC_2: now also PAD3.P; no longer T1.5
- net N$18: now also PAD2.P; no longer T1.1
- net N$45: now also PAD1.P; no longer T1.4
Changed lines of the file:
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@@
 <part name="GND20" library="SparkFun-Aesthetics" deviceset="GND" device=""/>
 <part name="J3" library="my-conn" deviceset="703W-00/54" device=""/>
-<part name="T1" library="my-transformers" deviceset="TR-LP30-1600" device=""/>
 <part name="B1" library="rectifier" deviceset="GBU4" device=""/>
 <part name="F1" library="fuse" deviceset="SH22,5" device=""/>
@@
 <part name="R24" library="SparkFun-Resistors" deviceset="RESISTOR" device="PTH-1/4W" value="5.1k"/>
 <part name="GND23" library="SparkFun-Aesthetics" deviceset="GND" device=""/>
+<part name="PAD1" library="wirepad" deviceset="3,81/1,4" device=""/>
+<part name="PAD2" library="wirepad" deviceset="3,81/1,4" device=""/>
+<part name="PAD3" library="wirepad" deviceset="3,81/1,4" device=""/>
+<part name="PAD4" library="wirepad" deviceset="3,81/1,4" device=""/>
 </parts>
 <sheets>
@@
 <instance part="J3" gate="L" x="50.8" y="210.82"/>
 <instance part="J3" gate="N" x="50.8" y="187.96"/>
-<instance part="T1" gate="G$1" x="104.14" y="200.66"/>
 <instance part="B1" gate="1" x="142.24" y="198.12"/>
 <instance part="F1" gate="1" x="63.5" y="210.82"/>
@@
 <instance part="GND41" gate="1" x="337.82" y="134.62"/>
 <instance part="LOGO1" gate="G$1" x="271.78" y="5.08"/>
+<instance part="PAD1" gate="1" x="99.06" y="213.36" rot="R180"/>
+<instance part="PAD2" gate="1" x="99.06" y="187.96" rot="R180"/>
+<instance part="PAD3" gate="1" x="109.22" y="213.36"/>
+<instance part="PAD4" gate="1" x="109.22" y="187.96"/>
 </instances>
 <busses>
@@
 </segment>
 </net>
-<net name="N$6" class="0">
-<segment>
-<pinref part="T1" gate="G$1" pin="3"/>
-<wire x1="96.52" y1="203.2" x2="93.98" y2="203.2" width="0.1524" layer="91"/>
-<wire x1="93.98" y1="203.2" x2="93.98" y2="198.12" width="0.1524" layer="91"/>
-<pinref part="T1" gate="G$1" pin="2"/>
-<wire x1="93.98" y1="198.12" x2="96.52" y2="198.12" width="0.1524" layer="91"/>
-</segment>
-</net>
-<net name="N$9" class="0">
-<segment>
-<pinref part="T1" gate="G$1" pin="6"/>
-<wire x1="111.76" y1="203.2" x2="114.3" y2="203.2" width="0.1524" layer="91"/>
-<wire x1="114.3" y1="203.2" x2="114.3" y2="198.12" width="0.1524" layer="91"/>
-<pinref part="T1" gate="G$1" pin="7"/>
-<wire x1="114.3" y1="198.12" x2="111.76" y2="198.12" width="0.1524" layer="91"/>
-</segment>
-</net>
 <net name="N$18" class="0">
 <segment>
 <pinref part="J3" gate="N" pin="P$1"/>
-<pinref part="T1" gate="G$1" pin="1"/>
 <wire x1="53.34" y1="187.96" x2="96.52" y2="187.96" width="0.1524" layer="91"/>
+<pinref part="PAD2" gate="1" pin="P"/>
 </segment>
 </net>
@@
 <segment>
 <pinref part="S1" gate="G$1" pin="O"/>
-<pinref part="T1" gate="G$1" pin="4"/>
 <wire x1="81.28" y1="213.36" x2="96.52" y2="213.36" width="0.1524" layer="91"/>
+<pinref part="PAD1" gate="1" pin="P"/>
 </segment>
 </net>
 <net name="AC_2" class="0">
 <segment>
-<pinref part="T1" gate="G$1" pin="5"/>
 <pinref part="B1" gate="1" pin="AC1"/>
 <wire x1="111.76" y1="213.36" x2="142.24" y2="213.36" width="0.1524" layer="91"/>
@@
 <junction x="142.24" y="213.36"/>
 <label x="142.24" y="215.9" size="1.778" layer="95" rot="R90" xref="yes"/>
+<pinref part="PAD3" gate="1" pin="P"/>
 </segment>
 <segment>
@@
 <net name="AC_1" class="0">
 <segment>
-<pinref part="T1" gate="G$1" pin="8"/>
 <pinref part="B1" gate="1" pin="AC2"/>
 <wire x1="111.76" y1="187.96" x2="142.24" y2="187.96" width="0.1524" layer="91"/>
@@
 <junction x="142.24" y="187.96"/>
 <label x="142.24" y="185.42" size="1.778" layer="95" rot="R270" xref="yes"/>
-</segment>
-<segment>
+<pinref part="PAD4" gate="1" pin="P"/>
+</segment>
+<segment>

Commit message: New board again
Parts:
- removed C30, C31: 47uF, my-cap:CAP_POLPTH-8/3.5
- removed F1: (no value), fuse:SH22,5
- removed J1: RCJ-21XXMILL, my:RCJ-21XXMILL
- removed J3: 703W-00/54, my-conn:703W-00/54
- removed PAD1, PAD2, PAD3, PAD4: (no value), wirepad:3,81/1,4
- removed S1: SW-M2012SA2W40, my-sw:SW-M2012SA2W40
- added Q22: KSP43, my-tran:KSP43
- added R46: 23.7k, SparkFun-Resistors:RESISTORPTH-1/4W
- added R47: 3.3k, SparkFun-Resistors:RESISTORPTH-1/4W
- added R48: 220, SparkFun-Resistors:RESISTORPTH-1/4W
- added X1: (no value), con-wago-508:W237-3E
- added X2: (no value), con-wago-508:W237-2N
- C10: value 470uF -> 1uF; device my-cap:CAP_POLPTH-12.5/5 -> capacitor-wima:C5/5
- C12, C2: value 0.1uF -> 1uF
- C13: value 1uF -> 0.33u; device capacitor-wima:C5/5 -> capacitor-wima:C5/7.2
- C14: value 0.33u -> 100uF; device capacitor-wima:C5/3.5 -> my-cap:CAP_POLPTH-8/3.5
- C15: value 10p -> 100uF; device SparkFun-Capacitors:CAPPTH -> my-cap:CAP_POLPTH-12.5/5
- C16, C6: device my-cap:CAP_POLPTH-8/3.5 -> my-cap:CAP_POLPTH-12.5/5
- C17, C18, C8: value 47uF -> 470uF; device my-cap:CAP_POLPTH-8/3.5 -> my-cap:CAP_POLPTH-12.5/5
- C19, C20: device my-cap:CAP_POLPTH-12.5/5 -> my-cap:CAP_POLPTH-18/7.5
- C21: value 470uF -> 4700uF; device my-cap:CAP_POLPTH-18/7.5 -> my-cap:CAP_POLSNAPIN-30/10
- C22: value 470uF -> 1uF; device my-cap:CAP_POLPTH-18/7.5 -> SparkFun-Capacitors:CAPPTH1
- C23: value 4700uF -> 47uF; device my-cap:CAP_POLSNAPIN-30/10 -> my-cap:CAP_POLPTH-12/5
- C24: value 1uF -> 10uF; device SparkFun-Capacitors:CAPPTH -> my-cap:CAP_POLPTH-5/2.5
- C25: value 47uF -> 10uF; device my-cap:CAP_POLPTH-12/5 -> my-cap:CAP_POLPTH-6.5/2.5
- C26: value 10uF -> 1uF; device my-cap:CAP_POLPTH-5/2.5 -> SparkFun-Capacitors:CAPPTH
- C27: value 10uF -> 1uF; device my-cap:CAP_POLPTH-6.5/2.5 -> SparkFun-Capacitors:CAPPTH
- C28, C29: value 1uF -> 47uF; device SparkFun-Capacitors:CAPPTH -> my-cap:CAP_POLPTH-8/3.5
- C4: device capacitor-wima:C5/3.5 -> capacitor-wima:C5/7.2
- C5: value 10p -> 100uF; device SparkFun-Capacitors:CAPPTH -> my-cap:CAP_POLPTH-8/3.5
- C7: value 47uF -> 100uF; device my-cap:CAP_POLPTH-8/3.5 -> my-cap:CAP_POLPTH-12.5/5
- IC3, IC4: value LM317MABT-OUT -> LM317MABT; device my-reg:LM317MABT-OUT -> my-reg:LM317MABT
- R10, R30: value 2.2k -> 4.7k
- R12, R31: value 10k -> 2.2k
- R13: value 4.7k -> 10k
- R14: value 10k -> 4.7k; device SparkFun-Electromechanical:TRIMPOT3362U-2 -> SparkFun-Resistors:RESISTORPTH-1/4W
- R15, R35: value 220 -> 10k; device SparkFun-Resistors:RESISTORPTH-1/4W -> SparkFun-Electromechanical:TRIMPOT3362U-2
- R17, R36, R37: value 2.2 -> 220
- R19, R38: value 2.2k -> 2.2
- R20: value 1Meg -> 2.2k
- R21: value 2Meg -> 1Meg
- R23: value 330 -> 2Meg
- R24: value 5.1k -> 1Meg
- R25, R6: value 1Meg -> 330
- R27: value 820 -> 5.1k
- R28: value 4.7k -> 330
- R29: value 2.2k -> 820
- R32: value 4.7k -> 2.2k
- R33: device SparkFun-Electromechanical:TRIMPOT3362U-2 -> SparkFun-Resistors:RESISTORPTH-1/4W
- R34: value 220 -> 4.7k
- R39: value 0.51 -> 2.2; device my-res:RESISTORPTH-1/2W -> SparkFun-Resistors:RESISTORPTH-1/4W
- R4: value 330 -> 1Meg
- R41: value 240 -> 0.51; device SparkFun-Resistors:RESISTORPTH-1/4W -> my-res:RESISTORPTH-1/2W
- R42: value 5.49k -> 2.2k
- R43: value 510 -> 240
- R44: value 23.7k -> 5.49k
- R45: value 3.3k -> 510
- R5: value 5.1k -> 330
- R7: value 330 -> 5.1k
- R8: value 820 -> 330
- R9: value 4.7k -> 820
- V1: device my-tubes:6DJ8-P-HORIZONTAL -> my-tubes:6DJ8-P21MM-BASE
Connections:
- removed net N$40: F1.1, J3L.P$1
- removed net N$44: F1.2, S1.P
- removed net N$45: PAD1.P, S1.O
- new net N$6: R5.1, V1A.TG
- new net N$9: R25.1, V1B.TG
- net +6.3FIL: now also R41.2, V1".H1; no longer R39.2, V1HEATER.H1
- net +LV: now also C21.+; no longer C23.+
- net AC_1: now also X2-2.KL; no longer PAD4.P
- net AC_2: now also C19.-, X2-1.KL; no longer C21.-, PAD3.P
- net CAT_L: now also R10.2; no longer R8.2
- net CAT_R: now also R29.2, R30.2; no longer R27.2, R28.2
- net FB_L: now also C5.-, C8.+, R18.1, R19.2; no longer C10.+, C6.-, R17.1, R18.2
- net FB_R: now also C14.-, C17.+, C18.+, R21.2, R38.1, R39.2; no longer C16.-, C19.+, C20.+, R20.2, R36.1, R37.2
- net FGND: now also V1".H3; no longer V1HEATER.H2
- net GND: now also C10.1, C15.-, C16.-, C20.-, C21.-, C22.2, C24.-, C26.2, C27.2, C28.-, C29.-, C6.-, R12.1, R17.1, R20.1, R23.2, R29.1, R32.1, R37.1, R4.1, R40.1, R46.2, R7.1, R9.1, X1-2.KL; no longer C11.1, C17.-, C18.-, C22.-, C24.2, C26.-, C27.-, C28.2, C29.2, C30.-, C31.-, C8.-, J1A.S, J1B.S, R11.1, R16.1, R19.1, R22.2, R25.1, R30.1, R35.1, R38.1, R42.2, R5.1, R6.1, R8.1, V1GNDPLANE.GND
- net G_L: now also R4.2, R5.2; no longer R6.2, V1A.TG
- net G_R: now also C13.2, R24.2; no longer C14.2, V1B.TG
- net HT: now also C15.+, C29.+, C6.+, R11.2, R28.2, R31.2, R45.1, R6.2, R8.2; no longer C17.+, C31.+, C7.+, R10.2, R23.2, R29.2, R4.2, R43.1, R7.2
- net IN_L: now also VR1A.S; no longer VR1B.S
- net IN_L*: now also VR1A.E, X1-3.KL; no longer J1B.T, VR1B.E
- net IN_R: now also C13.1, VR1B.S; no longer C14.1, VR1A.S
- net IN_R*: now also VR1B.E, X1-1.KL; no longer J1A.T, VR1A.E
- net N$10: now also R14.2, R15.CW; no longer R13.2, R14.CW
- net N$11: now also R18.2; no longer R17.2
- net N$12: now also R12.2, R15.CCW, R15.WIPER; no longer R11.2, R14.CCW, R14.WIPER
- net N$13: now also R19.1; no longer R18.1
- net N$14: now also R16.1; no longer R15.1
- net N$15: now also R17.2; no longer R16.2
- net N$16: now also R28.1; no longer R26.1
- net N$18: now also Q21.B, Q22.E, R48.2; no longer J3N.P$1, PAD2.P
- net N$19: now also C14.+, R30.1; no longer C16.+, R28.1
- net N$2: now also R8.1; no longer R7.1
- net N$20: now also R31.1; no longer R29.1
- net N$21: now also R33.2; no longer C15.2, R31.2
- net N$22: now also R33.1, R34.1; no longer R31.1, R32.1
- net N$23: now also R34.2, R35.CW; no longer R32.2, R33.CW
- net N$24: now also R32.2, R35.CCW, R35.WIPER; no longer R30.2, R33.CCW, R33.WIPER
- net N$25: now also R38.2; no longer R36.2
- net N$26: now also R39.1; no longer R37.1
- net N$27: now also R36.1; no longer R34.1
- net N$28: now also R37.2; no longer R35.2
- net N$3: now also R6.1; no longer R4.1
- net N$30: now also C24.+, C26.1, R43.2, R44.1; no longer C26.+, C28.1, R41.2, R42.1
- net N$31: now also C19.+; no longer C21.+
- net N$32: now also R41.1; no longer R39.1
- net N$33: now also C20.+, Q22.C, R42.1; no longer C22.+, R40.1
- net N$34: now also C22.1, C23.+, Q22.B, R42.2; no longer C24.1, C25.+, Q21.B, R40.2
- net N$36: now also C25.+, C27.1, R45.2, R46.1; no longer C27.+, C29.1, R43.2, R44.1
- net N$37: now also R48.1
- net N$39: now also R26.1; no longer R23.1
- net N$4: now also C5.+, R10.1; no longer C6.+, R9.1
- net N$41: now also C11.2, R23.1; no longer C13.2, R21.1
- net N$42: now also C10.2, R21.1; no longer C11.2, R20.1
- net N$43: now also C11.1; no longer C13.1
- net N$46: now also R47.2; no longer R45.2
- net N$47: now also R7.2; no longer R5.2
- net N$48: now also R27.2; no longer R24.2
- net N$5: now also R11.1; no longer R10.1
- net N$7: now also R13.2; no longer C5.2, R12.2
- net N$8: now also R14.1; no longer R12.1
- net OUT_L: now also C8.-, R20.2; no longer C10.-, R19.2
- net OUT_R: now also C17.-, C18.-, R40.2; no longer C19.-, C20.-, R38.2
- net PL_L: no longer C5.1
- net PL_R: no longer C15.1
- net VCC: now also C16.+, C28.+, C7.+, R16.2, R22.2, R36.2, R43.1, R47.1; no longer C18.+, C30.+, C8.+, R15.2, R21.2, R34.2, R41.1, R45.1
